File: 04_Electronics/joint_interface.kicad_pcb (KiCad board)
At the start: 4 copper layers, 100 x 100 mm, 48 parts, among them J1 5V INPUT, J2 MCU 3V3 I/O, J3 ENCODER 3V3, J4 NC LIMIT, J5 3V3 DRIVE I/O, J6 RS485 BUS, J7 E-STOP AUX NC, U1 AP2112K-3.3, U2 LTC2850IS8

Commit message: Review engineering models and polish ASTER-6 component access
Parts:
- F1: value 0.25A hold -> MF-NSMF025X-2; footprint Fuse:Fuse_1206_3216Metric -> ASTER_Interface:PTC_Bourns_MF-NSMF025X_1206
Changed lines of the file:
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@@
 		(embedded_fonts no)
 	)
-	(footprint "Fuse:Fuse_1206_3216Metric"
+	(footprint "ASTER_Interface:PTC_Bourns_MF-NSMF025X_1206"
 		(layer "F.Cu")
 		(at 35 32)
-		(descr "Fuse SMD 1206 (3216 Metric), square (rectangular) end terminal, IPC-7351 nominal, (Body size source: http://www.tortai-tech.com/upload/download/2011102023233369053.pdf)")
-		(tags "fuse")
+		(descr "Bourns MF-NSMF025X-2 PTC; manufacturer recommended nominal pads, mf-nsmf.pdf page 8. Body drawing is nominal; courtyard covers maximum body and pads.")
+		(tags "PTC polyfuse Bourns MF-NSMF025X 1206")
 		(property "Reference" "F1"
 			(at 0 -2.4 0)
@@
 			)
 		)
-		(property "Value" "0.25A hold"
-			(at 0 1.83 0)
+		(property "Value" "MF-NSMF025X-2"
+			(at 0 1.8 0)
 			(layer "F.Fab")
 			(hide yes)
@@
 			)
 		)
-		(property "Datasheet" ""
+		(property "Datasheet" "https://www.bourns.com/docs/product-datasheets/mf-nsmf.pdf"
 			(at 0 0 0)
 			(layer "F.Fab")
@@
 			)
 		)
-		(property "KiLib_Generator" "SMD_2terminal_chip_molded"
-			(at 0 0 0)
-			(layer "F.SilkS")
-			(hide yes)
-			(effects
-				(font
-					(size 1 1)
-					(thickness 0.15)
-				)
-			)
-		)
 		(attr smd)
 		(duplicate_pad_numbers_are_jumpers no)
 		(fp_line
-			(start -0.602064 -0.91)
-			(end 0.602064 -0.91)
+			(start -0.65 -1.03)
+			(end 0.65 -1.03)
 			(stroke
 				(width 0.12)
@@
 		)
 		(fp_line
-			(start -0.602064 0.91)
-			(end 0.602064 0.91)
+			(start -0.65 1.03)
+			(end 0.65 1.03)
 			(stroke
 				(width 0.12)
@@
 		)
 		(fp_rect
-			(start -2.28 -1.13)
-			(end 2.28 1.13)
+			(start -2.25 -1.15)
+			(end 2.25 1.15)
 			(stroke
 				(width 0.05)
@@
 			)
 		)
-		(pad "1" smd roundrect
-			(at -1.4 0)
-			(size 1.25 1.75)
+		(pad "1" smd rect
+			(at -1.5 0)
+			(size 1 1.6)
 			(layers "F.Cu" "F.Mask" "F.Paste")
-			(roundrect_rratio 0.2)
 			(net "/+5V_IN")
 		)
-		(pad "2" smd roundrect
-			(at 1.4 0)
-			(size 1.25 1.75)
+		(pad "2" smd rect
+			(at 1.5 0)
+			(size 1 1.6)
 			(layers "F.Cu" "F.Mask" "F.Paste")
-			(roundrect_rratio 0.2)
 			(net "/+5V_FUSED")
 		)
 		(embedded_fonts no)
-		(model "${KICAD10_3DMODEL_DIR}/Fuse.3dshapes/Fuse_1206_3216Metric.step"
-			(offset
-				(xyz 0 0 0)
-			)
-			(scale
-				(xyz 1 1 1)
-			)
-			(rotate
-				(xyz 0 0 0)
-			)
-		)
 	)
 	(footprint "Diode_SMD:D_SOD-123F"

Commit message: Rename the complete digital engineering project to INDRBT
Parts:
- F1: footprint ASTER_Interface:PTC_Bourns_MF-NSMF025X_1206 -> INDRBT_Interface:PTC_Bourns_MF-NSMF025X_1206
Other:
- board text added: "INDRBT JOINT / SENSOR INTERFACE"
- board text removed: "ASTER-6 JOINT / SENSOR INTERFACE"
Changed lines of the file:
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@@
 		(embedded_fonts no)
 	)
-	(footprint "ASTER_Interface:PTC_Bourns_MF-NSMF025X_1206"
+	(footprint "INDRBT_Interface:PTC_Bourns_MF-NSMF025X_1206"
 		(layer "F.Cu")
 		(at 35 32)
@@
 		)
 	)
-	(gr_text "ASTER-6  JOINT / SENSOR INTERFACE"
+	(gr_text "INDRBT  JOINT / SENSOR INTERFACE"
 		(at 69 24 0)
 		(layer "F.SilkS")
